File: pcb/kicad/pocket-chance-board.kicad_sch (KiCad schematic)
At the start: 124 parts, among them J1 SWD, J2 USB4085-GF-A, J3 LiPo JST-PH 2.0mm (pin 1 = + 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, J4 LCD 1.54in ST7789 module, JST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, J5 Speaker JST-PH, J6 microSD Molex 104031-0811, J7 STEMMA QT, J8 Expansion, Q1 FS8205A, Q2 DMG2305UX, SW1 BOOT, SW10 JOY LEFT, SW11 JOY RIGHT, SW12 JOY PRESS, SW2 RESET, SW3 POWER PCM12, SW4 A, SW5 B, SW6 X, SW7 Y, SW8 JOY UP, SW9 JOY DOWN, U1 RP2350A, U10 LSM6DSOXTR, U11 RM2, U2 W25Q128JVSIQ, U3 APS6404L-3SQR-SN, U4 USBLC6-2SC6, U5 BQ24074RGTR, U6 TPS63001DRCR, U7 DW01A, U8 PAM8302AASCR, U9 DS3231MZ+, Y1 12MHz ABM8-272-T3

Commit message: Buttons: 12 mm PTS125 (nearest standard size to John's 10 mm); fallback rows in PARTS.md
Co-Authored-By: Claude Fable 5.1 <noreply@anthropic.com>
Parts:
- SW4: value A -> A PTS125SM43SMTR2LFS; footprint Button_Switch_SMD:SW_SPST_PTS645Sx43SMTR92 -> Button_Switch_SMD:SW_Push_1P1T_NO_CK_PTS125Sx43SMTR
- SW5: value B -> B PTS125SM43SMTR2LFS; footprint Button_Switch_SMD:SW_SPST_PTS645Sx43SMTR92 -> Button_Switch_SMD:SW_Push_1P1T_NO_CK_PTS125Sx43SMTR
- SW6: value X -> X PTS125SM43SMTR2LFS; footprint Button_Switch_SMD:SW_SPST_PTS645Sx43SMTR92 -> Button_Switch_SMD:SW_Push_1P1T_NO_CK_PTS125Sx43SMTR
- SW7: value Y -> Y PTS125SM43SMTR2LFS; footprint Button_Switch_SMD:SW_SPST_PTS645Sx43SMTR92 -> Button_Switch_SMD:SW_Push_1P1T_NO_CK_PTS125Sx43SMTR
Changed lines of the file:
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@@
 			)
 		)
-		(property "Value" "A"
+		(property "Value" "A PTS125SM43SMTR2LFS"
 			(at 482.6 132.08 0)
 			(effects
@@
 			)
 		)
-		(property "Footprint" "Button_Switch_SMD:SW_SPST_PTS645Sx43SMTR92"
+		(property "Footprint" "Button_Switch_SMD:SW_Push_1P1T_NO_CK_PTS125Sx43SMTR"
 			(at 480.06 129.54 0)
 			(effects
@@
 			)
 		)
-		(property "Value" "B"
+		(property "Value" "B PTS125SM43SMTR2LFS"
 			(at 502.92 132.08 0)
 			(effects
@@
 			)
 		)
-		(property "Footprint" "Button_Switch_SMD:SW_SPST_PTS645Sx43SMTR92"
+		(property "Footprint" "Button_Switch_SMD:SW_Push_1P1T_NO_CK_PTS125Sx43SMTR"
 			(at 500.38 129.54 0)
 			(effects
@@
 			)
 		)
-		(property "Value" "X"
+		(property "Value" "X PTS125SM43SMTR2LFS"
 			(at 521.97 132.08 0)
 			(effects
@@
 			)
 		)
-		(property "Footprint" "Button_Switch_SMD:SW_SPST_PTS645Sx43SMTR92"
+		(property "Footprint" "Button_Switch_SMD:SW_Push_1P1T_NO_CK_PTS125Sx43SMTR"
 			(at 519.43 129.54 0)
 			(effects
@@
 			)
 		)
-		(property "Value" "Y"
+		(property "Value" "Y PTS125SM43SMTR2LFS"
 			(at 542.29 132.08 0)
 			(effects
@@
 			)
 		)
-		(property "Footprint" "Button_Switch_SMD:SW_SPST_PTS645Sx43SMTR92"
+		(property "Footprint" "Button_Switch_SMD:SW_Push_1P1T_NO_CK_PTS125Sx43SMTR"
 			(at 539.75 129.54 0)
 			(effects
