File: pcb/kicad/pocket-chance-board.kicad_sch (KiCad schematic)
At the start: 124 parts, among them J1 SWD, J2 USB4085-GF-A, J3 LiPo JST-PH 2.0mm (pin 1 = + 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, J4 LCD 1.54in ST7789 module, JST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, J5 Speaker JST-PH, J6 microSD Molex 104031-0811, J7 STEMMA QT, J8 Expansion, Q1 FS8205A, Q2 DMG2305UX, SW1 BOOT, SW10 JOY LEFT, SW11 JOY RIGHT, SW12 JOY PRESS, SW2 RESET, SW3 POWER PCM12, SW4 A PTS125SM43SMTR2LFS, SW5 B PTS125SM43SMTR2LFS, SW6 X PTS125SM43SMTR2LFS, SW7 Y PTS125SM43SMTR2LFS, SW8 JOY UP, SW9 JOY DOWN, U1 RP2350A, U10 LSM6DSOXTR, U11 RM2, U2 W25Q128JVSIQ, U3 APS6404L-3SQR-SN, U4 USBLC6-2SC6, U5 BQ24074RGTR, U6 TPS63001DRCR, U7 DW01A, U8 PAM8302AASCR, U9 DS3231MZ+, Y1 12MHz ABM8-272-T3

Commit message: Datasheet pass 1: charger values confirmed (EN table, K_ISET, TS, ITERM open, TMR), amplifier is the SO-8 part, PSRAM package confirmed
Parts:
- removed R17: 1.5k, Resistor_SMD:R_0402_1005Metric, symbol Device:R
- removed U8: PAM8302AASCR, Package_SO:SOIC-8_3.9x4.9mm_P1.27mm, symbol Amplifier_Audio:PAM8302AAS
- added U8: PAM8302AADCR, Package_SO:SOIC-8_3.9x4.9mm_P1.27mm, symbol Amplifier_Audio:PAM8302AAD
Connections:
- net +3V3: now also U8.1 (~{SD}), U8.6 (VDD)
- net AUDIO_INN: now also U8.4 (IN-)
- net AUDIO_INP: now also U8.3 (IN+)
- net GND: now also U8.7 (GND)
- net SPK+: now also U8.5 (OUT+)
- net SPK-: now also U8.8 (OUT-)
- net ITERM: no longer names the net of U5.15 (ITERM)
- no-connect marks 19 -> 20
