File: pcb/kicad/pocket-chance-board.kicad_pcb (KiCad board)
At the start: 2 copper layers, 0 parts

Commit message: Layout: first placement draft (150 x 100 mm, 4 layers), generated from the netlist by gen_pcb.py
All 132 footprints placed with nets; DRC: no overlaps or clearance errors, only silkscreen
cosmetics and the unrouted connections. Schematic unchanged (rev 0.10).
Parts:
- added BT2: CR1220, Battery:BatteryHolder_Keystone_3001_1x12mm, F.Cu at (65.0, 140.5)
- added C1: 100nF, Capacitor_SMD:C_0402_1005Metric, F.Cu at (116.0, 113.5)
- added C10: 100nF, Capacitor_SMD:C_0402_1005Metric, F.Cu at (115.2, 120.6)
- added C11: 10uF, Capacitor_SMD:C_0603_1608Metric, F.Cu at (154.0, 116.5)
- added C12: 2.2uF, Capacitor_SMD:C_0603_1608Metric, F.Cu at (128.5, 127.5)
- added C13: 4.7uF, Capacitor_SMD:C_0402_1005Metric, F.Cu at (132.6, 123.0)
- added C14: 4.7uF, Capacitor_SMD:C_0402_1005Metric, F.Cu at (132.6, 124.6)
- added C15: 4.7uF, Capacitor_SMD:C_0402_1005Metric, F.Cu at (132.6, 127.8)
- added C16: 15pF, Capacitor_SMD:C_0402_1005Metric, F.Cu at (107.5, 120.3)
- added C17: 15pF, Capacitor_SMD:C_0402_1005Metric, F.Cu at (107.5, 123.7)
- added C18: 100nF, Capacitor_SMD:C_0402_1005Metric, F.Cu at (138.0, 117.5)
- added C19: 100nF, Capacitor_SMD:C_0402_1005Metric, F.Cu at (146.0, 117.5)
- added C2: 100nF, Capacitor_SMD:C_0402_1005Metric, F.Cu at (118.4, 113.5)
- added C20: 1uF, Capacitor_SMD:C_0603_1608Metric, F.Cu at (167.0, 134.0)
- added C21: 10uF, Capacitor_SMD:C_0603_1608Metric, F.Cu at (158.0, 134.0)
- added C22: 10uF, Capacitor_SMD:C_0603_1608Metric, F.Cu at (162.0, 144.0)
- added C23: 10uF 16V X5R, Capacitor_SMD:C_0805_2012Metric, F.Cu at (156.0, 124.0)
- added C24: 100nF, Capacitor_SMD:C_0402_1005Metric, F.Cu at (156.0, 120.0)
- added C25: 10uF 10V X5R, Capacitor_SMD:C_0805_2012Metric, F.Cu at (160.0, 116.5)
- added C26: 10uF 10V X5R, Capacitor_SMD:C_0805_2012Metric, F.Cu at (163.6, 116.5)
- added C27: 100nF, Capacitor_SMD:C_0402_1005Metric, F.Cu at (184.0, 129.2)
- added C28: 100nF, Capacitor_SMD:C_0402_1005Metric, F.Cu at (146.6, 140.0)
- added C29: 10nF, Capacitor_SMD:C_0402_1005Metric, F.Cu at (84.4, 124.5)
- added C3: 100nF, Capacitor_SMD:C_0402_1005Metric, F.Cu at (120.8, 113.5)
- added C30: 1uF, Capacitor_SMD:C_0603_1608Metric, F.Cu at (86.8, 124.5)
- added C31: 1uF, Capacitor_SMD:C_0603_1608Metric, F.Cu at (89.2, 124.5)
- added C32: 10uF, Capacitor_SMD:C_0603_1608Metric, F.Cu at (94.0, 126.0)
- added C33: 10uF, Capacitor_SMD:C_0603_1608Metric, F.Cu at (70.0, 111.0)
- added C34: 100nF, Capacitor_SMD:C_0402_1005Metric, F.Cu at (90.5, 115.5)
- added C35: 100nF, Capacitor_SMD:C_0402_1005Metric, F.Cu at (90.5, 117.1)
- added C36: 100nF, Capacitor_SMD:C_0402_1005Metric, F.Cu at (98.0, 119.0)
- added C37: 100nF, Capacitor_SMD:C_0402_1005Metric, F.Cu at (98.0, 120.6)
- added C38: 10uF, Capacitor_SMD:C_0603_1608Metric, F.Cu at (110.0, 136.0)
- added C39: 100nF, Capacitor_SMD:C_0402_1005Metric, F.Cu at (110.0, 138.0)
- added C4: 100nF, Capacitor_SMD:C_0402_1005Metric, F.Cu at (125.5, 113.5)
- added C40: 4.7uF, Capacitor_SMD:C_0402_1005Metric, F.Cu at (132.6, 126.2)
- added C41: 1uF, Capacitor_SMD:C_0603_1608Metric, F.Cu at (94.0, 128.0)
- added C42: 1uF, Capacitor_SMD:C_0603_1608Metric, F.Cu at (94.0, 135.6)
- added C5: 100nF, Capacitor_SMD:C_0402_1005Metric, F.Cu at (127.9, 113.5)
- added C6: 100nF, Capacitor_SMD:C_0402_1005Metric, F.Cu at (128.0, 116.0)
- added C7: 100nF, Capacitor_SMD:C_0402_1005Metric, F.Cu at (128.0, 118.4)
- added C8: 100nF, Capacitor_SMD:C_0402_1005Metric, F.Cu at (115.2, 115.8)
- added C9: 100nF, Capacitor_SMD:C_0402_1005Metric, F.Cu at (115.2, 118.2)
- added D1: CHG, LED_SMD:LED_0603_1608Metric, F.Cu at (154.0, 136.0)
- added D2: USER, LED_SMD:LED_0603_1608Metric, F.Cu at (116.0, 131.0)
- added F1: MF-MSMF150/16X-2 1.5A, Fuse:Fuse_1812_4532Metric, F.Cu at (186.0, 145.5)
- added J1: SWD, Connector_PinHeader_1.27mm:PinHeader_2x05_P1.27mm_Vertical_SMD, F.Cu at (102.0, 130.0)
- added J2: USB4085-GF-A, Connector_USB:USB_C_Receptacle_GCT_USB4085, F.Cu at (174.0, 143.4)
- added J3: LiPo JST-PH 2.0mm (1 = + RED WIRE, 2 = -), Connector_JST:JST_PH_S2B-PH-SM4-TB_1x02-1MP_P2.00mm_Horizontal, F.Cu at (194.5, 138.0)
- added J4: LCD 1.54in ST7789 module, JST-PH 8-pin, Connector_JST:JST_PH_S8B-PH-SM4-TB_1x08-1MP_P2.00mm_Horizontal, F.Cu at (125.0, 102.0)
- added J5: Speaker JST-PH, Connector_JST:JST_PH_S2B-PH-SM4-TB_1x02-1MP_P2.00mm_Horizontal, F.Cu at (55.6, 128.0)
- added J6: microSD Molex 104031-0811, Connector_Card:microSD_HC_Molex_104031-0811, F.Cu at (57.6, 112.0)
- added J7: STEMMA QT, Connector_JST:JST_SH_SM04B-SRSS-TB_1x04-1MP_P1.00mm_Horizontal, F.Cu at (100.0, 145.5)
- added J8: Expansion (6 = VBAT_SENSE ADC node, not free GPIO), Connector_PinHeader_2.54mm:PinHeader_1x06_P2.54mm_Vertical, F.Cu at (80.0, 147.0)
- added JP2: RTC INT to GP14 (open; close only after firmware sets IMU I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, Jumper:SolderJumper-2_P1.3mm_Open_Pad1.0x1.5mm, F.Cu at (77.0, 124.0)
- added L1: 3.3uH AOTA-B201610S3R3-101-T, pcb_custom:AOTA-B201610S, F.Cu at (130.0, 125.0)
- added L2: 2.2uH ASPIAIG-F4020-2R2M, Inductor_SMD:L_Abracon_ASPIAIG-F4020, F.Cu at (166.0, 122.0)
- added Q1: FS8205A, Package_SO:TSSOP-8_4.4x3mm_P0.65mm, F.Cu at (190.0, 125.0)
- added Q3: AO3400A, Package_TO_SOT_SMD:SOT-23, F.Cu at (145.0, 136.0)
- added Q4: AO3401A, Package_TO_SOT_SMD:SOT-23, F.Cu at (140.0, 136.0)
- added R1: 200R, Resistor_SMD:R_0402_1005Metric, F.Cu at (125.5, 127.5)
- added R10: 27R, Resistor_SMD:R_0402_1005Metric, F.Cu at (154.0, 129.0)
- added R11: 27R, Resistor_SMD:R_0402_1005Metric, F.Cu at (154.0, 130.6)
- added R12: 10k, Resistor_SMD:R_0402_1005Metric, F.Cu at (156.0, 142.0)
- added R13: 10k, Resistor_SMD:R_0402_1005Metric, F.Cu at (167.0, 131.0)
- added R14: 1.8k, Resistor_SMD:R_0402_1005Metric, F.Cu at (158.2, 142.0)
- added R15: 3.0k, Resistor_SMD:R_0402_1005Metric, F.Cu at (160.4, 142.0)
- added R16: 68k, Resistor_SMD:R_0402_1005Metric, F.Cu at (162.6, 142.0)
- added R18: 1k, Resistor_SMD:R_0402_1005Metric, F.Cu at (154.0, 138.2)
- added R19: 100k, Resistor_SMD:R_0402_1005Metric, F.Cu at (168.0, 116.5)
- added R2: 33R, Resistor_SMD:R_0402_1005Metric, F.Cu at (132.6, 129.4)
- added R20: 470R, Resistor_SMD:R_0402_1005Metric, F.Cu at (184.0, 126.0)
- added R21: 2k, Resistor_SMD:R_0402_1005Metric, F.Cu at (184.0, 127.6)
- added R22: 0R, Resistor_SMD:R_0603_1608Metric, F.Cu at (184.0, 141.0)
- added R23: 100k, Resistor_SMD:R_0402_1005Metric, F.Cu at (142.2, 140.0)
- added R24: 100k, Resistor_SMD:R_0402_1005Metric, F.Cu at (144.4, 140.0)
- added R25: 1k, Resistor_SMD:R_0402_1005Metric, F.Cu at (82.0, 124.5)
- added R26: 10k, Resistor_SMD:R_0402_1005Metric, F.Cu at (67.0, 105.5)
- added R27: 10k, Resistor_SMD:R_0402_1005Metric, F.Cu at (67.0, 107.1)
- added R28: 10k, Resistor_SMD:R_0402_1005Metric, F.Cu at (67.0, 108.7)
- added R29: 10k, Resistor_SMD:R_0402_1005Metric, F.Cu at (67.0, 110.3)
- added R3: 1k, Resistor_SMD:R_0402_1005Metric, F.Cu at (114.0, 125.8)
- added R30: 10k, Resistor_SMD:R_0402_1005Metric, F.Cu at (67.0, 111.9)
- added R31: 4.7k, Resistor_SMD:R_0402_1005Metric, F.Cu at (84.0, 116.0)
- added R32: 4.7k, Resistor_SMD:R_0402_1005Metric, F.Cu at (84.0, 117.6)
- added R33: 470R, Resistor_SMD:R_0402_1005Metric, F.Cu at (126.5, 131.0)
- added R34: 10k, Resistor_SMD:R_0402_1005Metric, F.Cu at (128.9, 131.0)
- added R35: 1k, Resistor_SMD:R_0402_1005Metric, F.Cu at (119.0, 131.0)
- added R36: 5.6k, Resistor_SMD:R_0402_1005Metric, F.Cu at (134.0, 136.0)
- added R37: 10k, Resistor_SMD:R_0402_1005Metric, F.Cu at (134.0, 137.6)
- added R39: 100k, Resistor_SMD:R_0402_1005Metric, F.Cu at (140.0, 140.0)
- added R4: 10k, Resistor_SMD:R_0402_1005Metric, F.Cu at (134.0, 106.5)
- added R42: 10k, Resistor_SMD:R_0402_1005Metric, F.Cu at (77.0, 120.0)
- added R43: 1k, Resistor_SMD:R_0402_1005Metric, F.Cu at (77.0, 122.0)
- added R44: 47k, Resistor_SMD:R_0402_1005Metric, F.Cu at (94.0, 134.0)
- added R5: 1k, Resistor_SMD:R_0402_1005Metric, F.Cu at (136.4, 106.5)
- added R6: 10k, Resistor_SMD:R_0402_1005Metric, F.Cu at (149.0, 106.5)
- added R7: 10k, Resistor_SMD:R_0402_1005Metric, F.Cu at (114.0, 128.0)
- added R8: 5.1k, Resistor_SMD:R_0402_1005Metric, F.Cu at (166.0, 142.0)
- added R9: 5.1k, Resistor_SMD:R_0402_1005Metric, F.Cu at (166.0, 143.6)
- added SW1: BOOT, Button_Switch_SMD:SW_SPST_PTS645Sx43SMTR92, F.Cu at (109.5, 111.5)
- added SW10: DPAD LEFT PTS645SM43SMTR92, Button_Switch_SMD:SW_SPST_PTS645Sx43SMTR92, F.Cu at (60.0, 88.0)
- added SW11: DPAD RIGHT PTS645SM43SMTR92, Button_Switch_SMD:SW_SPST_PTS645Sx43SMTR92, F.Cu at (88.0, 88.0)
- added SW12: DPAD PRESS PTS645SM43SMTR92, Button_Switch_SMD:SW_SPST_PTS645Sx43SMTR92, F.Cu at (74.0, 88.0)
- added SW2: RESET, Button_Switch_SMD:SW_SPST_PTS645Sx43SMTR92, F.Cu at (90.0, 110.0)
- added SW3: POWER PCM12, Button_Switch_SMD:SW_SPDT_PCM12, F.Cu at (196.5, 120.0)
- added SW4: A PTS125SM43SMTR2LFS, Button_Switch_SMD:SW_Push_1P1T_NO_CK_PTS125Sx43SMTR, F.Cu at (190.0, 86.0)
- added SW5: B PTS125SM43SMTR2LFS, Button_Switch_SMD:SW_Push_1P1T_NO_CK_PTS125Sx43SMTR, F.Cu at (172.0, 102.0)
- added SW6: X PTS125SM43SMTR2LFS, Button_Switch_SMD:SW_Push_1P1T_NO_CK_PTS125Sx43SMTR, F.Cu at (172.0, 70.0)
- added SW7: Y PTS125SM43SMTR2LFS, Button_Switch_SMD:SW_Push_1P1T_NO_CK_PTS125Sx43SMTR, F.Cu at (154.0, 86.0)
- added SW8: DPAD UP PTS645SM43SMTR92, Button_Switch_SMD:SW_SPST_PTS645Sx43SMTR92, F.Cu at (74.0, 75.0)
- added SW9: DPAD DOWN PTS645SM43SMTR92, Button_Switch_SMD:SW_SPST_PTS645Sx43SMTR92, F.Cu at (74.0, 101.0)
- added TP1: VBUS, TestPoint:TestPoint_Pad_D1.5mm, F.Cu at (182.0, 138.0)
- added TP2: VSYS, TestPoint:TestPoint_Pad_D1.5mm, F.Cu at (154.0, 146.0)
- added TP3: +3V3, TestPoint:TestPoint_Pad_D1.5mm, F.Cu at (150.0, 120.0)
- added TP4: 1V1, TestPoint:TestPoint_Pad_D1.5mm, F.Cu at (136.0, 130.0)
- added TP5: GND, TestPoint:TestPoint_Pad_D1.5mm, F.Cu at (107.0, 139.0)
- added TP6: GND, TestPoint:TestPoint_Pad_D1.5mm, F.Cu at (196.0, 146.0)
- added TP7: BAT+, TestPoint:TestPoint_Pad_D1.5mm, F.Cu at (178.0, 130.0)
- added TP8: RUN, TestPoint:TestPoint_Pad_D1.5mm, F.Cu at (108.0, 126.0)
- added U1: RP2350A, Package_DFN_QFN:QFN-60-1EP_7x7mm_P0.4mm_EP3.4x3.4mm, F.Cu at (122.0, 120.0)
- added U10: LSM6DSOXTR, Package_LGA:LGA-14_3x2.5mm_P0.5mm_LayoutBorder3x4y, F.Cu at (94.0, 116.0)
- added U11: RM2, pcb_custom:RM2, F.Cu at (122.0, 141.8)
- added U2: W25Q128JVSIQ, Package_SO:SOIC-8_5.3x5.3mm_P1.27mm, F.Cu at (138.0, 112.0)
- added U3: APS6404L-3SQR-SN, Package_SO:SOIC-8_3.9x4.9mm_P1.27mm, F.Cu at (146.0, 112.0)
- added U4: USBLC6-2SC6, Package_TO_SOT_SMD:SOT-23-6, F.Cu at (174.0, 136.0)
- added U5: BQ24074RGTR, Package_DFN_QFN:VQFN-16-1EP_3x3mm_P0.5mm_EP1.68x1.68mm_ThermalVias, F.Cu at (162.0, 138.0)
- added U6: TPS63001DRCR, Package_SON:Texas_DRC0010J_ThermalVias, F.Cu at (160.0, 122.0)
- added U7: DW01A, Package_TO_SOT_SMD:SOT-23-6, F.Cu at (190.0, 130.0)
- added U8: PAM8302AADCR, Package_SO:SOIC-8_3.9x4.9mm_P1.27mm, F.Cu at (88.0, 130.0)
- added U9: DS3231MZ+, Package_SO:SOIC-8_3.9x4.9mm_P1.27mm, F.Cu at (70.0, 116.0)
- added Y1: 12MHz ABM8-272-T3, Crystal:Crystal_SMD_3225-4Pin_3.2x2.5mm, F.Cu at (111.0, 122.0)
Other:
- board outline added: 150 x 100 mm
- copper layers 2 -> 4
- board text added: "Pocket Chance spin 1 rev 0.10 placement draft"
- board text added: "SCREEN MODULE (1.54in, on standoffs, cable to J4)"
