File: pcb/kicad/pocket-chance-board.kicad_pcb (KiCad board)
At the start: 4 copper layers, 150 x 100 mm, 138 parts, among them J1 SWD, J2 USB4085-GF-A, J3 LiPo JST-PH 2.0mm (1 = + RED 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, J4 LCD 1.54in ST7789 module, JST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, J5 Speaker JST-PH, J6 microSD Molex 104031-0811, J7 STEMMA QT, J8 Expansion (6 = VBAT_SENSE ADC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, Q1 FS8205A, Q3 AO3400A, Q4 AO3401A, SW1 BOOT, SW10 DPAD LEFT PTS645SM43SMTR92, SW11 DPAD RIGHT PTS645SM43SMTR92, SW12 DPAD PRESS PTS645SM43SMTR92, SW2 RESET, SW3 POWER PCM12, SW4 A PTS125SM43SMTR2LFS, SW5 B PTS125SM43SMTR2LFS, SW6 X PTS125SM43SMTR2LFS, SW7 Y PTS125SM43SMTR2LFS, SW8 DPAD UP PTS645SM43SMTR92, SW9 DPAD DOWN PTS645SM43SMTR92, U1 RP2350A, U10 LSM6DSOXTR, U11 RM2, U2 W25Q128JVSIQ, U3 APS6404L-3SQR-SN, U4 USBLC6-2SC6, U5 BQ24074RGTR, U6 TPS63001DRCR, U7 DW01A, U8 PAM8302AADCR, U9 DS3231MZ+, Y1 12MHz ABM8-272-T3

Commit message: Rev 0.11 prep (NOT for merge until John's go): J9 1x8 2.54 mm screen header on J4's nets, pins named on silk
John's ruling (option B) via the PM. Netlist diff vs pcb-design: only J9 added, on +3V3, GND, LCD_MOSI,
LCD_SCK, LCD_CS, LCD_DC, LCD_RST, LCD_BL. ERC 0 errors, 2 expected warnings. Placed between the screen
reserve and J4 at y 44; DRC: no placement errors. The rest of rev 0.11 (probe pads, F1 footprint,
ADC cap) waits for John.

Co-Authored-By: Claude Opus 5.5 <noreply@anthropic.com>
Parts:
- added J9: LCD header 2.54 mm (wire by name; one screen at a time), Connector_PinHeader_2.54mm:PinHeader_1x08_P2.54mm_Vertical, F.Cu at (116.1, 94.0)
Other:
- board text added: "3V3"
- board text added: "BL"
- board text added: "CS"
- board text added: "DC"
- board text added: "GND"
- board text added: "J9: WIRE BY NAME, MODULES DIFFER IN ORDER. ONE SCREEN AT A TIME"
- board text added: "MOSI/SDA"
- board text added: "RST"
- board text added: "SCK/SCL"

Commit message: Rev 0.11 (John's 'yes all'): J9 screen header, probe pads TP9-TP14, F1 Bourns footprint, C43 ADC 100 nF, backlight link R49 with unfitted Q6/R50/R51
- GPIO13 now net LCD_BL_CTL, joined to LCD_BL by R49 0 ohm (fitted): behaviour unchanged
- Q6 AO3401A high-side switch + R50 1k + R51 100k DNP, for a direct-drive BL module (then BL active LOW)
- netlist diff vs rev 0.10: 12 parts added, F1 footprint field changed, LCD_BL split; nothing removed
- ERC 0 errors, 2 expected warnings; 144 parts placed; placement DRC clean

Co-Authored-By: Claude Opus 5.5 <noreply@anthropic.com>
Parts:
- added C43: 100nF, Capacitor_SMD:C_0402_1005Metric, F.Cu at (123.2, 127.8)
- added Q6: AO3401A (DNP: fit only for a direct-drive BL module), Package_TO_SOT_SMD:SOT-23, F.Cu at (143.0, 101.5)
- added R49: 0R, Resistor_SMD:R_0402_1005Metric, F.Cu at (143.0, 97.0)
- added R50: 1k, Resistor_SMD:R_0402_1005Metric, F.Cu at (147.0, 101.5)
- added R51: 100k, Resistor_SMD:R_0402_1005Metric, F.Cu at (147.0, 103.2)
- added TP10: CELL_F, TestPoint:TestPoint_Pad_D1.5mm, F.Cu at (187.6, 141.6)
- added TP11: SDA, TestPoint:TestPoint_Pad_D1.5mm, F.Cu at (80.5, 114.0)
- added TP12: SCL, TestPoint:TestPoint_Pad_D1.5mm, F.Cu at (80.5, 110.5)
- added TP13: SD_SCK, TestPoint:TestPoint_Pad_D1.5mm, F.Cu at (67.0, 117.0)
- added TP14: LCD_SCK, TestPoint:TestPoint_Pad_D1.5mm, F.Cu at (138.5, 96.0)
- added TP9: CELL_P, TestPoint:TestPoint_Pad_D1.5mm, F.Cu at (184.0, 141.6)
- F1: footprint Fuse:Fuse_1812_4532Metric -> pcb_custom:Fuse_Bourns_MF-MSMF_1812
- moved R22 3.16 mm to (181.0, 140.0)
Connections:
- U1 pad 17: LCD_BL -> LCD_BL_CTL
Other:
- board text added: "Pocket Chance spin 1 rev 0.11 placement draft"
- board text added: "Q6 FITTED = BL ACTIVE LOW (then remove R49)"
- board text removed: "Pocket Chance spin 1 rev 0.10 placement draft"
